Commit message: Fix xacro tutorial model

File: gazebo_tutorials/src/xacro_tutorial/model/links.xacro (robot description, xacro)
@@ -64,5 +64,5 @@
         <!-- Joint -->
         <joint name="${link}_joint" type="revolute">
-            <origin xyz="0.0 0.0 ${width/2+heigth/2}" rpy="0.0 0.0 0.0"/>
+            <origin xyz="0.0 0.0 ${heigth}" rpy="0.0 0.0 0.0"/>
             <parent link="${link}_tail"/>
             <child link="${link}_head"/>

File: gazebo_tutorials/src/xacro_tutorial/model/unibot.urdf (robot description, URDF)
Before this commit: robot unibot, 15 links, 14 joints
Joints:
- joint a1_joint: origin xyz=0.0 0.0 0.35 rpy=0.0 0.0 0.0 -> xyz=0.0 0.0 0.5 rpy=0.0 0.0 0.0
- joint a2_joint: origin xyz=0.0 0.0 0.35 rpy=0.0 0.0 0.0 -> xyz=0.0 0.0 0.5 rpy=0.0 0.0 0.0
- joint a3_joint: origin xyz=0.0 0.0 0.35 rpy=0.0 0.0 0.0 -> xyz=0.0 0.0 0.5 rpy=0.0 0.0 0.0
- joint a4_joint: origin xyz=0.0 0.0 0.35 rpy=0.0 0.0 0.0 -> xyz=0.0 0.0 0.5 rpy=0.0 0.0 0.0
- joint a5_joint: origin xyz=0.0 0.0 0.35 rpy=0.0 0.0 0.0 -> xyz=0.0 0.0 0.5 rpy=0.0 0.0 0.0
- joint a6_joint: origin xyz=0.0 0.0 0.35 rpy=0.0 0.0 0.0 -> xyz=0.0 0.0 0.5 rpy=0.0 0.0 0.0
- joint a7_joint: origin xyz=0.0 0.0 0.35 rpy=0.0 0.0 0.0 -> xyz=0.0 0.0 0.5 rpy=0.0 0.0 0.0
