Commit message: commit current state

File: gazebo_tutorials/src/xacro_tutorial/model/unibot.xacro (robot description, xacro)
@@ -1,22 +1,65 @@
 <?xml version="1.0"?>
 <robot name="unibot" xmlns:xacro="http://www.ros.org/wiki/xacro">
-    <!-- Includes -->
-    <xacro:include filename="$(find xacro_tutorial)/model/links.xacro"/>
-    <xacro:include filename="$(find xacro_tutorial)/model/union.xacro"/>
-    <!-- Links -->
-    <xacro:unit link="a1"/>
-    <xacro:unit link="a2"/>
-    <xacro:unit link="a3"/>
-    <xacro:unit link="a4"/>
-    <xacro:unit link="a5"/>
-    <xacro:unit link="a6"/>
-    <xacro:unit link="a7"/>
-    <xacro:pin root_link="a1"/>
-    <!-- Joints -->
-    <xacro:union parent="a1" child="a2" y=" 1"/>
-    <xacro:union parent="a2" child="a3" x="-1"/>
-    <xacro:union parent="a3" child="a4" y="-1"/>
-    <xacro:union parent="a4" child="a5" x="-1"/>
-    <xacro:union parent="a5" child="a6" y="-1"/>
-    <xacro:union parent="a6" child="a7" x=" 1"/>
+  <!-- Includes -->
+  <xacro:include filename="$(find xacro_tutorial)/model/links.xacro"/>
+  <xacro:include filename="$(find xacro_tutorial)/model/union.xacro"/>
+  <!-- Links -->
+  <xacro:unit link="a1"/>
+  <xacro:unit link="a2"/>
+  <xacro:unit link="a3"/>
+  <xacro:unit link="a4"/>
+  <xacro:unit link="a5"/>
+  <xacro:unit link="a6"/>
+  <xacro:unit link="a7"/>
+  <xacro:pin root_link="a1"/>
+  <!-- Joints -->
+  <xacro:union parent="a1" child="a2" y=" 1"/>
+  <xacro:union parent="a2" child="a3" x="-1"/>
+  <xacro:union parent="a3" child="a4" y="-1"/>
+  <xacro:union parent="a4" child="a5" x="-1"/>
+  <xacro:union parent="a5" child="a6" y="-1"/>
+  <xacro:union parent="a6" child="a7" x=" 1"/>
+  <gazebo>
+  <!-- <transmission name="tran1">
+      <type>transmission_interface/SimpleTransmission</type>
+      <joint name="a1_joint">
+        <hardwareInterface>EffortJointInterface</hardwareInterface>
+      </joint>
+      <actuator name="motor1">
+        <hardwareInterface>EffortJointInterface</hardwareInterface>
+        <mechanicalReduction>1</mechanicalReduction>
+      </actuator>
+    </transmission> -->
+    <!-- <transmission name="tran1">
+      <type>transmission_interface/SimpleTransmission</type>
+      <joint name="a1_joint">
+        <hardwareInterface>EffortJointInterface</hardwareInterface>
+      </joint>
+      <actuator name="motor1">
+        <hardwareInterface>EffortJointInterface</hardwareInterface>
+        <mechanicalReduction>1</mechanicalReduction>
+      </actuator>
+    </transmission> -->
+    <plugin name="gazebo_ros_control" filename="libgazebo_ros_control.so">
+        <robotSimType>gazebo_ros_control/DefaultRobotHWSim</robotSimType>
+    </plugin>
+    <plugin name=   "gazebo_ros_joint_state_publisher"
+        filename="libgazebo_ros_joint_state_publisher.so">
+      <update_rate>100</update_rate>
+      <joint_name>a1_joint</joint_name>
+      <joint_name>a2_joint</joint_name>
+    </plugin>
+  </gazebo>
+  <ros2_control name="test" type="actuator">
+    <hardware>
+    </hardware>
+    <joint name="a1_joint">
+      <command_interface name="position">
+        <param name="min">0</param>
+        <param name="max">50</param>
+      </command_interface>
+      <state_interface name="position"/>
+      <state_interface name="velocity"/>
+    </joint>
+  </ros2_control>
 </robot>

Commit message: change dir

File: gazebo_tutorials/src/xacro_tutorial/model/unibot.xacro (robot description, xacro)
@@ -2,46 +2,41 @@
 <robot name="unibot" xmlns:xacro="http://www.ros.org/wiki/xacro">
   <!-- Includes -->
-  <xacro:include filename="$(find xacro_tutorial)/model/links.xacro"/>
-  <xacro:include filename="$(find xacro_tutorial)/model/union.xacro"/>
+  <xacro:include filename="$(find xacro_tutorial)/model/xacro/links.xacro"/>
+  <xacro:include filename="$(find xacro_tutorial)/model/xacro/union.xacro"/>
   <!-- Links -->
   <xacro:unit link="a1"/>
   <xacro:unit link="a2"/>
-  <xacro:unit link="a3"/>
+  <!-- <xacro:unit link="a3"/>
   <xacro:unit link="a4"/>
   <xacro:unit link="a5"/>
   <xacro:unit link="a6"/>
-  <xacro:unit link="a7"/>
+  <xacro:unit link="a7"/> -->
   <xacro:pin root_link="a1"/>
   <!-- Joints -->
   <xacro:union parent="a1" child="a2" y=" 1"/>
-  <xacro:union parent="a2" child="a3" x="-1"/>
+  <!-- <xacro:union parent="a2" child="a3" x="-1"/>
   <xacro:union parent="a3" child="a4" y="-1"/>
   <xacro:union parent="a4" child="a5" x="-1"/>
   <xacro:union parent="a5" child="a6" y="-1"/>
-  <xacro:union parent="a6" child="a7" x=" 1"/>
+  <xacro:union parent="a6" child="a7" x=" 1"/> -->
+  <ros2_control name="test" type="system">
+    <hardware>
+      <plugin>gazebo_ros2_control/GazeboSystem</plugin>
+    </hardware>
+    <joint name="a1_joint">
+      <command_interface name="effort">
+        <param name="min">-100000</param>
+        <param name="max">100000</param>
+      </command_interface>
+      <state_interface name="position"/>
+      <state_interface name="velocity"/>
+      <state_interface name="effort"/>
+    </joint>
+  </ros2_control>
   <gazebo>
-  <!-- <transmission name="tran1">
-      <type>transmission_interface/SimpleTransmission</type>
-      <joint name="a1_joint">
-        <hardwareInterface>EffortJointInterface</hardwareInterface>
-      </joint>
-      <actuator name="motor1">
-        <hardwareInterface>EffortJointInterface</hardwareInterface>
-        <mechanicalReduction>1</mechanicalReduction>
-      </actuator>
-    </transmission> -->
-    <!-- <transmission name="tran1">
-      <type>transmission_interface/SimpleTransmission</type>
-      <joint name="a1_joint">
-        <hardwareInterface>EffortJointInterface</hardwareInterface>
-      </joint>
-      <actuator name="motor1">
-        <hardwareInterface>EffortJointInterface</hardwareInterface>
-        <mechanicalReduction>1</mechanicalReduction>
-      </actuator>
-    </transmission> -->
-    <plugin name="gazebo_ros_control" filename="libgazebo_ros_control.so">
-        <robotSimType>gazebo_ros_control/DefaultRobotHWSim</robotSimType>
-    </plugin>
+    <plugin name="gazebo_ros2_control" filename="libgazebo_ros2_control.so"></plugin>
+    <robot_sim_type>gazebo_ros2_control/GazeboSystem</robot_sim_type>
+  </gazebo>
+  <!-- <gazebo>
     <plugin name=   "gazebo_ros_joint_state_publisher"
         filename="libgazebo_ros_joint_state_publisher.so">
@@ -50,16 +45,4 @@
       <joint_name>a2_joint</joint_name>
     </plugin>
-  </gazebo>
-  <ros2_control name="test" type="actuator">
-    <hardware>
-    </hardware>
-    <joint name="a1_joint">
-      <command_interface name="position">
-        <param name="min">0</param>
-        <param name="max">50</param>
-      </command_interface>
-      <state_interface name="position"/>
-      <state_interface name="velocity"/>
-    </joint>
-  </ros2_control>
+  </gazebo> -->
 </robot>

File: gazebo_tutorials/src/xacro_tutorial/model/xacro/links.xacro (robot description, xacro)
@@ -1,5 +1,5 @@
 <?xml version="1.0"?>
 <robot xmlns:xacro="http://www.ros.org/wiki/xacro">
-    <xacro:include filename="$(find xacro_tutorial)/model/properties.xacro"/>
+    <xacro:include filename="$(find xacro_tutorial)/model/xacro/properties.xacro"/>
     <xacro:macro name="unit" params="link">
         <!-- Geometry Macros-->

File: gazebo_tutorials/src/xacro_tutorial/model/xacro/union.xacro (robot description, xacro)
@@ -1,5 +1,5 @@
 <robot xmlns:xacro="http://www.ros.org/wiki/xacro">
     <xacro:macro name="union" params="parent child x=0 y=0 z=0">
-        <xacro:include filename="$(find xacro_tutorial)/model/properties.xacro"/>
+        <xacro:include filename="$(find xacro_tutorial)/model/xacro/properties.xacro"/>
         <joint name="${parent}_${child}_joint" type="fixed">
             <origin xyz="${x*width/2} ${y*width/2} ${z*width/2+width/2}"

Commit message: commit current state

File: gazebo_tutorials/src/xacro_tutorial/model/unibot.xacro (robot description, xacro)
@@ -20,5 +20,5 @@
   <xacro:union parent="a5" child="a6" y="-1"/>
   <xacro:union parent="a6" child="a7" x=" 1"/> -->
-  <ros2_control name="test" type="system">
+  <ros2_control name="GazeboSystem" type="system">
     <hardware>
       <plugin>gazebo_ros2_control/GazeboSystem</plugin>
@@ -35,6 +35,7 @@
   </ros2_control>
   <gazebo>
-    <plugin name="gazebo_ros2_control" filename="libgazebo_ros2_control.so"></plugin>
-    <robot_sim_type>gazebo_ros2_control/GazeboSystem</robot_sim_type>
+    <plugin filename="libgazebo_ros2_control.so" name="gazebo_ros2_control">
+      <parameters>$(find xacro_tutorial)/config/controllers.yaml</parameters>
+    </plugin>
   </gazebo>
   <!-- <gazebo>

File: gazebo_tutorials/src/xacro_tutorial/model/xacro/links.xacro (robot description, xacro)
@@ -68,5 +68,5 @@
             <child link="${link}_head"/>
             <axis xyz="0.0 0.0 1.0"/>
-            <limit lower="${-pi/2}" upper="${pi/2}" effort="1000000" velocity="1000000"/>
+            <limit lower="${-2*pi}" upper="${2*pi}" effort="1000000" velocity="1000000"/>
         </joint>
     </xacro:macro>
