Commit message: update current state

File: gazebo_tutorials/ros2_control_tutorial/model/unibot.urdf (robot description, URDF)
Before this commit: robot unibot, 15 links, 14 joints
Links:
- removed link a3_head
- removed link a3_tail
- removed link a4_head
- removed link a4_tail
- removed link a5_head
- removed link a5_tail
- removed link a6_head
- removed link a6_tail
- removed link a7_head
- removed link a7_tail
Joints:
- removed joint a2_a3_joint
- removed joint a3_a4_joint
- removed joint a3_joint
- removed joint a4_a5_joint
- removed joint a4_joint
- removed joint a5_a6_joint
- removed joint a5_joint
- removed joint a6_a7_joint
- removed joint a6_joint
- removed joint a7_joint
- joint a1_joint: limit lower=-1.5707963267948966 upper=1.5707963267948966 effort=1000000 velocity=1000000 -> lower=-6.283185307179586 upper=6.283185307179586 effort=1000000 velocity=1000000; type revolute -> continuous
- joint a2_joint: limit lower=-1.5707963267948966 upper=1.5707963267948966 effort=1000000 velocity=1000000 -> lower=-6.283185307179586 upper=6.283185307179586 effort=1000000 velocity=1000000; type revolute -> continuous

File: gazebo_tutorials/ros2_control_tutorial/model/unibot.xacro (robot description, xacro)
@@ -2,21 +2,13 @@
 <robot name="unibot" xmlns:xacro="http://www.ros.org/wiki/xacro">
   <!-- Includes -->
-  <xacro:include filename="$(find xacro_tutorial)/model/xacro/links.xacro"/>
-  <xacro:include filename="$(find xacro_tutorial)/model/xacro/union.xacro"/>
+  <xacro:include filename="$(find ros2_control_tutorial)/model/xacro/links.xacro"/>
+  <xacro:include filename="$(find ros2_control_tutorial)/model/xacro/union.xacro"/>
   <!-- Links -->
   <xacro:unit link="a1"/>
   <xacro:unit link="a2"/>
-  <xacro:unit link="a3"/>
-  <xacro:unit link="a4"/>
-  <xacro:unit link="a5"/>
-  <xacro:unit link="a6"/>
-  <xacro:unit link="a7"/>
   <xacro:pin root_link="a1"/>
   <!-- Joints -->
   <xacro:union parent="a1" child="a2" y=" 1"/>
-  <xacro:union parent="a2" child="a3" x="-1"/>
-  <xacro:union parent="a3" child="a4" y="-1"/>
-  <xacro:union parent="a4" child="a5" x="-1"/>
-  <xacro:union parent="a5" child="a6" y="-1"/>
-  <xacro:union parent="a6" child="a7" x=" 1"/>
+  <!-- Plugin -->
+  <xacro:include filename="$(find ros2_control_tutorial)/model/xacro/plugins.xacro"/>
 </robot>

File: gazebo_tutorials/ros2_control_tutorial/model/xacro/links.xacro (robot description, xacro)
@@ -1,5 +1,5 @@
 <?xml version="1.0"?>
 <robot xmlns:xacro="http://www.ros.org/wiki/xacro">
-    <xacro:include filename="$(find xacro_tutorial)/model/xacro/properties.xacro"/>
+    <xacro:include filename="$(find ros2_control_tutorial)/model/xacro/properties.xacro"/>
     <xacro:macro name="unit" params="link">
         <!-- Geometry Macros-->
@@ -63,5 +63,5 @@
         </gazebo>
         <!-- Joint -->
-        <joint name="${link}_joint" type="revolute">
+        <joint name="${link}_joint" type="continuous">
             <origin xyz="0.0 0.0 ${heigth}" rpy="0.0 0.0 0.0"/>
             <parent link="${link}_tail"/>

File: gazebo_tutorials/ros2_control_tutorial/model/xacro/union.xacro (robot description, xacro)
@@ -1,5 +1,5 @@
 <robot xmlns:xacro="http://www.ros.org/wiki/xacro">
     <xacro:macro name="union" params="parent child x=0 y=0 z=0">
-        <xacro:include filename="$(find xacro_tutorial)/model/xacro/properties.xacro"/>
+        <xacro:include filename="$(find ros2_control_tutorial)/model/xacro/properties.xacro"/>
         <joint name="${parent}_${child}_joint" type="fixed">
             <origin xyz="${x*width/2} ${y*width/2} ${z*width/2+width/2}"
