Commit message: to 6DOF

File: mypkg/xacro/myrobot_description.urdf.xacro (robot description, xacro)
@@ -2,113 +2,151 @@
 <robot xmlns:xacro="http://www.ros.org/wiki/xacro">
   <xacro:macro name="myrobot_description" params="parent">
-  <!-- Constants for robot dimensions -->
-  <xacro:property name="mass" value="1" /> <!-- arbitrary value for mass -->
-  <xacro:property name="width" value="0.1" /> <!-- Square dimensions (widthxwidth) of beams -->
-  <xacro:property name="height1" value="2" /> <!-- Link 1 -->
-  <xacro:property name="height2" value="1" /> <!-- Link 2 -->
-  <xacro:property name="height3" value="1" /> <!-- Link 3 -->
-  <xacro:property name="axel_offset" value="0.05" /> <!-- Space btw top of beam and the each joint -->
-  <!-- Base Link -->
   <link name="base_link">
+    <visual>
+      <geometry>
+        <box size="0.1 0.1 0.1"/>
+      </geometry>
+      <material name = "">
+        <color rgba="0.8 0.8 0.8 1.0"/>
+      </material>
+    </visual>
     <collision>
-      <origin xyz="0 0 ${height1/2}" rpy="0 0 0"/>
       <geometry>
-        <box size="${width} ${width} ${height1}"/>
+        <box size="0.1 0.1 0.1"/>
       </geometry>
     </collision>
+  </link>
+  <link name="link1">
     <visual>
-      <origin xyz="0 0 ${height1/2}" rpy="0 0 0"/>
       <geometry>
-        <box size="${width} ${width} ${height1}"/>
+        <box size="0.2 0.1 0.1"/>
       </geometry>
-      <material name="orange">
-        <color rgba="${255/255} ${108/255} ${10/255} 1.0"/>
+      <material name = "">
+        <color rgba="0.8 0.8 0.8 1.0"/>
       </material>
     </visual>
-    <inertial>
-      <origin xyz="0 0 ${height1/2}" rpy="0 0 0"/>
-      <mass value="${mass}"/>
-      <inertia
-        ixx="${mass / 12.0 * (width*width + height1*height1)}" ixy="0.0" ixz="0.0"
-        iyy="${mass / 12.0 * (height1*height1 + width*width)}" iyz="0.0"
-        izz="${mass / 12.0 * (width*width + width*width)}"/>
-    </inertial>
-  </link>
-  <joint name="joint1" type="continuous">
-    <parent link="base_link"/>
-    <child link="link1"/>
-    <origin xyz="0 ${width} ${height1 - axel_offset}" rpy="0 0 0"/>
-    <axis xyz="0 1 0"/>
-    <dynamics damping="0.7"/>
-    <limit effort="100" velocity="1.0"/>
-  </joint>
-  <!-- Middle Link -->
-  <link name="link1">
     <collision>
-      <origin xyz="0 0 ${height2/2 - axel_offset}" rpy="0 0 0"/>
       <geometry>
-        <box size="${width} ${width} ${height2}"/>
+        <box size="0.2 0.1 0.1"/>
       </geometry>
     </collision>
+  </link>
+  <link name="link2">
     <visual>
-      <origin xyz="0 0 ${height2/2 - axel_offset}" rpy="0 0 0"/>
       <geometry>
-        <box size="${width} ${width} ${height2}"/>
+        <box size="0.2 0.1 0.1"/>
       </geometry>
-      <material name="yellow">
-        <color rgba="1.0 1.0 0.0 1.0"/>
+      <material name = "">
+        <color rgba="0.8 0.8 0.8 1.0"/>
       </material>
     </visual>
-    <inertial>
-      <origin xyz="0 0 ${height2/2 - axel_offset}" rpy="0 0 0"/>
-      <mass value="${mass}"/>
-      <inertia
-        ixx="${mass / 12.0 * (width*width + height2*height2)}" ixy="0.0" ixz="0.0"
-        iyy="${mass / 12.0 * (height2*height2 + width*width)}" iyz="0.0"
-        izz="${mass / 12.0 * (width*width + width*width)}"/>
-    </inertial>
+    <collision>
+      <geometry>
+        <box size="0.2 0.1 0.1"/>
+      </geometry>
+    </collision>
   </link>
-  <joint name="joint2" type="continuous">
+  <link name="link3">
+    <visual>
+      <geometry>
+        <box size="0.2 0.1 0.1"/>
+      </geometry>
+      <material name = "">
+        <color rgba="0.8 0.8 0.8 1.0"/>
+      </material>
+    </visual>
+    <collision>
+      <geometry>
+        <box size="0.2 0.1 0.1"/>
+      </geometry>
+    </collision>
+  </link>
+  <link name="link4">
+    <visual>
+      <geometry>
+        <box size="0.2 0.1 0.1"/>
+      </geometry>
+      <material name = "">
+        <color rgba="0.8 0.8 0.8 1.0"/>
+      </material>
+    </visual>
+    <collision>
+      <geometry>
+        <box size="0.2 0.1 0.1"/>
+      </geometry>
+    </collision>
+  </link>
+  <link name="link5">
+    <visual>
+      <geometry>
+        <box size="0.2 0.1 0.1"/>
+      </geometry>
+      <material name = "">
+        <color rgba="0.8 0.8 0.8 1.0"/>
+      </material>
+    </visual>
+    <collision>
+      <geometry>
+        <box size="0.2 0.1 0.1"/>
+      </geometry>
+    </collision>
+  </link>
+  <link name="link6">
+    <visual>
+      <geometry>
+        <box size="0.1 0.1 0.1"/>
+      </geometry>
+      <material name = "">
+        <color rgba="0.8 0.8 0.8 1.0"/>
+      </material>
+    </visual>
+    <collision>
+      <geometry>
+        <box size="0.1 0.1 0.1"/>
+      </geometry>
+    </collision>
+  </link>
+  <joint name="joint1" type="revolute">
+    <origin xyz="0.0 0.0 0.1"/>
+    <axis xyz="0 0 1"/>
+    <parent link="${parent}"/>
+    <child link="link1"/>
+    <limit lower="-3.14159" upper="3.14159" effort="100" velocity="1.0"/>
+  </joint>
+  <joint name="joint2" type="revolute">
+    <origin xyz="0.2 0.0 0.0"/>
+    <axis xyz="0 0 1"/>
     <parent link="link1"/>
     <child link="link2"/>
-    <origin xyz="0 ${width} ${height2 - axel_offset*2}" rpy="0 0 0"/>
-    <axis xyz="0 1 0"/>
-    <dynamics damping="0.7"/>
-    <limit effort="100" velocity="1.0"/>
+    <limit lower="-3.14159" upper="3.14159" effort="100" velocity="1.0"/>
   </joint>
-  <!-- Top Link -->
-  <link name="link2">
-    <collision>
-      <origin xyz="0 0 ${height3/2 - axel_offset}" rpy="0 0 0"/>
-      <geometry>
-        <box size="${width} ${width} ${height3}"/>
-      </geometry>
-    </collision>
-    <visual>
-      <origin xyz="0 0 ${height3/2 - axel_offset}" rpy="0 0 0"/>
-      <geometry>
-        <box size="${width} ${width} ${height3}"/>
-      </geometry>
-      <material name="orange">
-        <color rgba="${255/255} ${108/255} ${10/255} 1.0"/>
-      </material>
-    </visual>
-    <inertial>
-      <origin xyz="0 0 ${height3/2 - axel_offset}" rpy="0 0 0"/>
-      <mass value="${mass}"/>
-      <inertia
-        ixx="${mass / 12.0 * (width*width + height3*height3)}" ixy="0.0" ixz="0.0"
-        iyy="${mass / 12.0 * (height3*height3 + width*width)}" iyz="0.0"
-        izz="${mass / 12.0 * (width*width + width*width)}"/>
-    </inertial>
-  </link>
-  <joint name="tool_joint" type="fixed">
-    <origin xyz="0 0 1" rpy="0 0 0" />
+  <joint name="joint3" type="revolute">
+    <origin xyz="0.2 0.0 0.0"/>
+    <axis xyz="0 0 1"/>
     <parent link="link2"/>
-    <child link="tool_link" />
+    <child link="link3"/>
+    <limit lower="-3.14159" upper="3.14159" effort="100" velocity="1.0"/>
   </joint>
-  <!-- Tool Link -->
-  <link name="tool_link">
-  </link>
+  <joint name="joint4" type="revolute">
+    <origin xyz="0.2 0.0 0.0"/>
+    <axis xyz="0 0 1"/>
+    <parent link="link3"/>
+    <child link="link4"/>
+    <limit lower="-3.14159" upper="3.14159" effort="100" velocity="1.0"/>
+  </joint>
+  <joint name="joint5" type="revolute">
+    <origin xyz="0.2 0.0 0.0"/>
+    <axis xyz="0 0 1"/>
+    <parent link="link4"/>
+    <child link="link5"/>
+    <limit lower="-3.14159" upper="3.14159" effort="100" velocity="1.0"/>
+  </joint>
+  <joint name="joint6" type="revolute">
+    <origin xyz="0.2 0.0 0.0"/>
+    <axis xyz="0 0 1"/>
+    <parent link="link5"/>
+    <child link="link6"/>
+    <limit lower="-3.14159" upper="3.14159" effort="100" velocity="1.0"/>
+  </joint>
   </xacro:macro>
 </robot>

File: mypkg/xacro/myrobot_ros2_control.xacro (robot description, xacro)
@@ -8,6 +8,6 @@
       <joint name="joint1">
         <command_interface name="position">
-          <param name="min">-1</param>
-          <param name="max">1</param>
+          <param name="min">-3</param>
+          <param name="max">3</param>
         </command_interface>
         <state_interface name="position"/>
@@ -15,6 +15,34 @@
       <joint name="joint2">
         <command_interface name="position">
-          <param name="min">-1</param>
-          <param name="max">1</param>
+          <param name="min">-3</param>
+          <param name="max">3</param>
+        </command_interface>
+        <state_interface name="position"/>
+      </joint>
+      <joint name="joint3">
+        <command_interface name="position">
+          <param name="min">-3</param>
+          <param name="max">3</param>
+        </command_interface>
+        <state_interface name="position"/>
+      </joint>
+      <joint name="joint4">
+        <command_interface name="position">
+          <param name="min">-3</param>
+          <param name="max">3</param>
+        </command_interface>
+        <state_interface name="position"/>
+      </joint>
+      <joint name="joint5">
+        <command_interface name="position">
+          <param name="min">-3</param>
+          <param name="max">3</param>
+        </command_interface>
+        <state_interface name="position"/>
+      </joint>
+      <joint name="joint6">
+        <command_interface name="position">
+          <param name="min">-3</param>
+          <param name="max">3</param>
         </command_interface>
         <state_interface name="position"/>

Commit message: update description

File: mypkg/xacro/myrobot_description.urdf.xacro (robot description, xacro)
@@ -2,151 +2,87 @@
 <robot xmlns:xacro="http://www.ros.org/wiki/xacro">
   <xacro:macro name="myrobot_description" params="parent">
-  <link name="base_link">
-    <visual>
-      <geometry>
-        <box size="0.1 0.1 0.1"/>
-      </geometry>
-      <material name = "">
-        <color rgba="0.8 0.8 0.8 1.0"/>
-      </material>
-    </visual>
-    <collision>
-      <geometry>
-        <box size="0.1 0.1 0.1"/>
-      </geometry>
-    </collision>
-  </link>
-  <link name="link1">
-    <visual>
-      <geometry>
-        <box size="0.2 0.1 0.1"/>
-      </geometry>
-      <material name = "">
-        <color rgba="0.8 0.8 0.8 1.0"/>
-      </material>
-    </visual>
-    <collision>
-      <geometry>
-        <box size="0.2 0.1 0.1"/>
-      </geometry>
-    </collision>
-  </link>
-  <link name="link2">
-    <visual>
-      <geometry>
-        <box size="0.2 0.1 0.1"/>
-      </geometry>
-      <material name = "">
-        <color rgba="0.8 0.8 0.8 1.0"/>
-      </material>
-    </visual>
-    <collision>
-      <geometry>
-        <box size="0.2 0.1 0.1"/>
-      </geometry>
-    </collision>
-  </link>
-  <link name="link3">
-    <visual>
-      <geometry>
-        <box size="0.2 0.1 0.1"/>
-      </geometry>
-      <material name = "">
-        <color rgba="0.8 0.8 0.8 1.0"/>
-      </material>
-    </visual>
-    <collision>
-      <geometry>
-        <box size="0.2 0.1 0.1"/>
-      </geometry>
-    </collision>
-  </link>
-  <link name="link4">
-    <visual>
-      <geometry>
-        <box size="0.2 0.1 0.1"/>
-      </geometry>
-      <material name = "">
-        <color rgba="0.8 0.8 0.8 1.0"/>
-      </material>
-    </visual>
-    <collision>
-      <geometry>
-        <box size="0.2 0.1 0.1"/>
-      </geometry>
-    </collision>
-  </link>
-  <link name="link5">
-    <visual>
-      <geometry>
-        <box size="0.2 0.1 0.1"/>
-      </geometry>
-      <material name = "">
-        <color rgba="0.8 0.8 0.8 1.0"/>
-      </material>
-    </visual>
-    <collision>
-      <geometry>
-        <box size="0.2 0.1 0.1"/>
-      </geometry>
-    </collision>
-  </link>
-  <link name="link6">
-    <visual>
-      <geometry>
-        <box size="0.1 0.1 0.1"/>
-      </geometry>
-      <material name = "">
-        <color rgba="0.8 0.8 0.8 1.0"/>
-      </material>
-    </visual>
-    <collision>
-      <geometry>
-        <box size="0.1 0.1 0.1"/>
-      </geometry>
-    </collision>
-  </link>
+  <!-- helper macro -->
+    <xacro:macro name="create_link" params="
+        link_name
+        xyz_offset
+        rpy_offset
+        box_size
+        ">
+    <link name="${link_name}">
+      <visual>
+        <origin xyz="${xyz_offset}" rpy="${rpy_offset}"/>
+        <geometry>
+          <box size="${box_size}"/>
+        </geometry>
+      </visual>
+      <collision>
+        <origin xyz="${xyz_offset}" rpy="${rpy_offset}"/>
+        <geometry>
+          <box size="${box_size}"/>
+        </geometry>
+      </collision>
+      <inertial>
+        <mass value="1"/>
+        <inertia ixx="1.0" ixy="0.0" ixz="0.0" iyy="1.0" iyz="0.0" izz="1.0"/>
+      </inertial>
+    </link>
+  </xacro:macro>
+  <!-- link definitions -->
+  <xacro:create_link link_name="base_link" xyz_offset="0 0 0" rpy_offset="0 0 0" box_size="0.2 0.2 0.2"/>
+  <xacro:create_link link_name="link1"     xyz_offset="0 0 0.075" rpy_offset="0 0 0" box_size="0.15 0.15 0.05"/>
+  <xacro:create_link link_name="link2"     xyz_offset="0.15 0 0" rpy_offset="0 0 0" box_size="0.3 0.1 0.1"/>
+  <xacro:create_link link_name="link3"     xyz_offset="0.25 0 0" rpy_offset="0 0 0" box_size="0.5 0.1 0.1"/>
+  <xacro:create_link link_name="link4"     xyz_offset="0.2 0 0" rpy_offset="0 0 0" box_size="0.4 0.1 0.1"/>
+  <xacro:create_link link_name="link5"     xyz_offset="0.1 0 0" rpy_offset="0 0 0" box_size="0.2 0.1 0.1"/>
+  <xacro:create_link link_name="link6"     xyz_offset="0.075 0 0" rpy_offset="0 0 0" box_size="0.15 0.1 0.1"/>
+  <link name="tool"/>
+  <!-- joints - main serial chain -->
   <joint name="joint1" type="revolute">
-    <origin xyz="0.0 0.0 0.1"/>
+    <parent link="base_link"/>
+    <child link="link1"/>
+    <origin xyz="0 0 0.061584" rpy="0 0 0"/>
     <axis xyz="0 0 1"/>
-    <parent link="${parent}"/>
-    <child link="link1"/>
-    <limit lower="-3.14159" upper="3.14159" effort="100" velocity="1.0"/>
+    <limit effort="1000.0" lower="${-pi}" upper="${pi}" velocity="2.5"/>
   </joint>
   <joint name="joint2" type="revolute">
-    <origin xyz="0.2 0.0 0.0"/>
-    <axis xyz="0 0 1"/>
     <parent link="link1"/>
     <child link="link2"/>
-    <limit lower="-3.14159" upper="3.14159" effort="100" velocity="1.0"/>
+    <origin xyz="-0.101717 0 0.182284" rpy="${-pi/2} -${pi/3} ${pi/2}"/>
+    <axis xyz="0 0 1"/>
+    <limit effort="1000.0" lower="${-pi}" upper="${pi}" velocity="2.5"/>
   </joint>
   <joint name="joint3" type="revolute">
-    <origin xyz="0.2 0.0 0.0"/>
-    <axis xyz="0 0 1"/>
     <parent link="link2"/>
     <child link="link3"/>
-    <limit lower="-3.14159" upper="3.14159" effort="100" velocity="1.0"/>
+    <origin xyz="0.685682 0 0.041861" rpy="0 ${pi} ${pi+pi/2}"/>
+    <axis xyz="0 0 1"/>
+    <limit effort="1000.0" lower="${-pi}" upper="${pi}" velocity="2.5"/>
   </joint>
   <joint name="joint4" type="revolute">
-    <origin xyz="0.2 0.0 0.0"/>
-    <axis xyz="0 0 1"/>
     <parent link="link3"/>
     <child link="link4"/>
-    <limit lower="-3.14159" upper="3.14159" effort="100" velocity="1.0"/>
+    <origin xyz="0.518777 0 0.067458" rpy="0 ${pi} ${pi+pi/6}"/>
+    <axis xyz="0 0 1"/>
+    <limit effort="1000.0" lower="${-pi}" upper="${pi}" velocity="2.5"/>
   </joint>
   <joint name="joint5" type="revolute">
-    <origin xyz="0.2 0.0 0.0"/>
-    <axis xyz="0 0 1"/>
     <parent link="link4"/>
     <child link="link5"/>
-    <limit lower="-3.14159" upper="3.14159" effort="100" velocity="1.0"/>
+    <origin xyz="0.112654 0 0.110903" rpy="${pi/2} ${pi} ${pi/2}"/>
+    <axis xyz="0 0 1"/>
+    <limit effort="1000.0" lower="${-pi}" upper="${pi}" velocity="2.5"/>
   </joint>
   <joint name="joint6" type="revolute">
-    <origin xyz="0.2 0.0 0.0"/>
-    <axis xyz="0 0 1"/>
     <parent link="link5"/>
     <child link="link6"/>
-    <limit lower="-3.14159" upper="3.14159" effort="100" velocity="1.0"/>
+    <origin xyz="-0.085976 0 0.133436" rpy="0 ${-pi/2} 0"/>
+    <axis xyz="0 0 1"/>
+    <limit effort="1000.0" lower="${-pi}" upper="${pi}" velocity="2.5"/>
   </joint>
-  </xacro:macro>
+  <joint name="joint-tool" type="fixed">
+    <parent link="link6"/>
+    <child link="tool"/>
+    <origin xyz="0 0 .185" rpy="0 0 0"/>
+  </joint>
+</xacro:macro>
 </robot>
